Commit message: fix urdf rover model (rockers and wheels)

File: src/rover_description/urdf/macros/rocker_assembly.xacro (robot description, xacro)
@@ -12,5 +12,7 @@
       </inertial>
       <visual>
-        <origin xyz="${rocker_mesh_align_xyz}" rpy="0 0 ${-pi / 2.0}"/>
+        <!-- rocker.stl is not a mirrored pair; the left one is yawed 180 deg so
+             the same mesh faces the right way on both sides. -->
+        <origin xyz="0 ${rocker_mesh_align_y_left if y_sign > 0 else rocker_mesh_align_y_right} 0" rpy="0 0 ${pi / 2.0 * y_sign}"/>
         <geometry>
           <mesh filename="package://rover_description/meshes/suspension/rocker.stl" scale="1 1 1"/>

File: src/rover_description/urdf/macros/wheel_assembly.xacro (robot description, xacro)
@@ -11,5 +11,5 @@
       </inertial>
       <visual>
-        <origin xyz="0 ${wheel_mount_hub_offset * y_sign} ${wheel_mount_visual_z}" rpy="0 0 0"/>
+        <origin xyz="0.001 ${wheel_mount_hub_offset * y_sign} ${wheel_mount_visual_z}" rpy="0 0 0"/>
         <geometry>
           <mesh filename="package://rover_description/meshes/suspension/wheel_mount.stl" scale="1 ${y_sign} 1"/>
@@ -28,5 +28,5 @@
       <parent link="${parent}"/>
       <child link="${prefix}_wheel_mount_link"/>
-      <origin xyz="${x_sign * (rocker_length / 2.0 - rocker_mount_x_offset)} ${rocker_hub_y} ${rocker_hub_z}" rpy="0 0 0"/>
+      <origin xyz="${x_sign * (rocker_length / 2.0 - rocker_mount_x_offset)} ${rocker_hub_y * y_sign} ${rocker_hub_z}" rpy="0 0 0"/>
       <axis xyz="0 0 1"/>
       <limit lower="${-steering_limit}" upper="${steering_limit}" effort="${steering_effort}" velocity="${steering_velocity}"/>

File: src/rover_description/urdf/properties.xacro (robot description, xacro)
@@ -23,10 +23,15 @@
   <xacro:property name="rocker_height" value="0.187"/>  <!-- Z -->
   <xacro:property name="rocker_mass" value="1.0"/>
-  <!-- Mesh alignment: centers rocker.stl on the rocker link's own origin -->
-  <xacro:property name="rocker_mesh_align_xyz" value="0 0.0001 0.0"/>
+  <!-- Mesh alignment: centers rocker.stl on the rocker link's own origin. The left
+       rocker's mesh is yawed 180 deg, so its Y correction is not a mirror of the right. -->
+  <xacro:property name="rocker_mesh_align_y_left" value="-0.02"/>
+  <xacro:property name="rocker_mesh_align_y_right" value="0.02"/>
   <!-- Wheel-mount attachment point: where the wheel_mount hub attaches to the rocker's end,
        relative to the rocker's pivot origin -->
+  <!-- Lateral offset stays 0: the steering axis and wheel centre sit on the rocker
+       pivot plane, so wheel centres land at +/-track_width/2, which is what
+       swerve_kinematics and the odometry in controllers.yaml assume. -->
   <xacro:property name="rocker_mount_x_offset" value="0.050"/>
-  <xacro:property name="rocker_hub_y" value="-0.0258"/>
+  <xacro:property name="rocker_hub_y" value="0.0"/>
   <xacro:property name="rocker_hub_z" value="-0.1140"/>
   <!-- ===================== WHEEL MOUNT (steering knuckle) ===================== -->
@@ -37,9 +42,9 @@
   <xacro:property name="wheel_mount_mass" value="0.162"/>
   <!-- Mesh alignment: centers wheel_mount.stl's steering bore on the link's own origin -->
-  <xacro:property name="wheel_mount_hub_offset" value="0.1253"/>
-  <xacro:property name="wheel_mount_visual_z" value="-0.1814"/>
+  <xacro:property name="wheel_mount_hub_offset" value="0.1489"/>
+  <xacro:property name="wheel_mount_visual_z" value="-0.1799"/>
   <!-- Wheel attachment point: axle position relative to the steering bore -->
   <xacro:property name="wheel_mount_drop" value="0.1857"/>
-  <xacro:property name="axle_lateral_offset" value="-0.0168"/>
+  <xacro:property name="axle_lateral_offset" value="0.0"/>
   <!-- ===================== WHEEL ===================== -->
   <!-- Geometry -->
