Commit message: partially fix

File: src/rover_description/urdf/macros/wheel_assembly.xacro (robot description, xacro)
@@ -41,7 +41,9 @@
       </inertial>
       <visual>
-        <origin xyz="0 ${wheel_hub_offset * y_sign} 0" rpy="0 0 0"/>
+        <!-- Right wheel is yawed 180 deg rather than scaled by -1: a negative
+             scale flips polygon winding, inverting the mesh normals. -->
+        <origin xyz="0 ${wheel_hub_offset * y_sign} 0" rpy="0 0 ${0 if y_sign > 0 else pi}"/>
         <geometry>
-          <mesh filename="package://rover_description/meshes/suspension/wheel.stl" scale="1 ${y_sign} 1"/>
+          <mesh filename="package://rover_description/meshes/suspension/wheel.stl" scale="1 1 1"/>
         </geometry>
         <material name="dark_wheel"/>

File: src/rover_description/urdf/properties.xacro (robot description, xacro)
@@ -71,6 +71,6 @@
   <xacro:property name="drive_velocity" value="10"/>
   <!-- ===================== WHEEL GROUND CONTACT FRICTION ===================== -->
-  <xacro:property name="wheel_mu1" value="1.0"/>
-  <xacro:property name="wheel_mu2" value="1.0"/>
+  <xacro:property name="wheel_mu1" value="1.2"/>
+  <xacro:property name="wheel_mu2" value="1.2"/>
   <xacro:property name="wheel_kp" value="1000000.0"/>
   <xacro:property name="wheel_kd" value="1.0"/>
