Commit message: feature: add parameter to remove stereo camera from urdf and rviz visualization

File: src/rover_description/urdf/rover.urdf.xacro (robot description, xacro)
@@ -99,15 +99,19 @@
   </joint>
   <!-- ===================== ZED2i STEREO CAMERA ===================== -->
-  <xacro:stereo_camera
-    use_sim="$(arg use_sim)"
-    simulate_rgb="$(arg stereo_camera_simulate_rgb)"
-    simulate_depth="$(arg stereo_camera_simulate_depth)"
-    simulate_imu="$(arg stereo_camera_simulate_imu)"
-  />
-  <joint name="zed2i_base_joint" type="fixed">
-    <parent link="main_body_link"/>
-    <child link="zed2i_camera_link"/>
-    <origin xyz="${zed2i_x} ${zed2i_y} ${zed2i_z}" rpy="${zed2i_rx} ${zed2i_ry} ${zed2i_rz}"/>
-  </joint>
+  <!-- Both the macro call and the joint are guarded: the joint's child link is
+       created by the macro, so neither can stand without the other. -->
+  <xacro:if value="$(arg use_stereo_camera)">
+    <xacro:stereo_camera
+      use_sim="$(arg use_sim)"
+      simulate_rgb="$(arg stereo_camera_simulate_rgb)"
+      simulate_depth="$(arg stereo_camera_simulate_depth)"
+      simulate_imu="$(arg stereo_camera_simulate_imu)"
+    />
+    <joint name="zed2i_base_joint" type="fixed">
+      <parent link="main_body_link"/>
+      <child link="zed2i_camera_link"/>
+      <origin xyz="${zed2i_x} ${zed2i_y} ${zed2i_z}" rpy="${zed2i_rx} ${zed2i_ry} ${zed2i_rz}"/>
+    </joint>
+  </xacro:if>
   <!-- ===================== RPLIDAR S2 ===================== -->
   <xacro:lidar

File: src/rover_description/urdf/rover.xacro (robot description, xacro)
@@ -12,4 +12,10 @@
        depends on) is namespaced. -->
   <xacro:arg name="rover_namespace" default="rover"/>
+  <!-- Set false to leave the ZED2i out of the model entirely: its links, its
+       joint to main_body_link, and the $(find zed_description) lookup that the
+       stereo_camera macro performs. Needed wherever the ZED ROS 2 wrapper
+       (which provides zed_description) is not installed, since xacro resolves
+       that package the moment the macro is instantiated. -->
+  <xacro:arg name="use_stereo_camera" default="true"/>
   <!-- Sensor Simulation Arguments -->
   <xacro:arg name="lidar_simulate_scan" default="false"/>
